Commit message: Configure KR 16 R2010-2 simulation model

File: src/foundation/pickcell_description/urdf/pickcell.urdf.xacro (robot description, xacro)
@@ -1,9 +1,17 @@
 <?xml version="1.0"?>
-<robot
-  xmlns:xacro="http://www.ros.org/wiki/xacro"
-  name="pickcell">
-  <!-- فریم مرجع کل سیستم -->
+<robot xmlns:xacro="http://www.ros.org/wiki/xacro" name="pickcell">
+  <!--
+    Cell description using the maintained ROS 2 model of the KUKA
+    KR 16 R2010-2. Robot dimensions, joint axes, joint limits and meshes live
+    in kuka_cybertech_support; they are intentionally not duplicated here.
+  -->
+  <xacro:include filename="$(find kuka_cybertech_support)/urdf/kr16_r2010_2_macro.xacro"/>
+  <xacro:arg name="robot_prefix" default=""/>
+  <xacro:arg name="robot_mount_xyz" default="0 0 0"/>
+  <xacro:arg name="robot_mount_rpy" default="0 0 0"/>
+  <xacro:arg name="tcp_xyz" default="0 0 0"/>
+  <xacro:arg name="tcp_rpy" default="0 0 0"/>
+  <xacro:property name="prefix" value="$(arg robot_prefix)"/>
   <link name="world"/>
-  <!-- فریم سلول صنعتی -->
   <link name="cell"/>
   <joint name="world_to_cell" type="fixed">
@@ -12,55 +20,26 @@
     <origin xyz="0 0 0" rpy="0 0 0"/>
   </joint>
-  <!-- محل نصب ربات -->
+  <!-- robot_base is the configurable mounting pose inside the cell. -->
   <link name="robot_base"/>
   <joint name="cell_to_robot_base" type="fixed">
     <parent link="cell"/>
     <child link="robot_base"/>
+    <origin xyz="$(arg robot_mount_xyz)" rpy="$(arg robot_mount_rpy)"/>
+  </joint>
+  <xacro:kuka_kr16_r2010_2_robot
+    prefix="${prefix}"
+    package_name="kuka_cybertech_support"/>
+  <joint name="robot_base_to_kuka_base_link" type="fixed">
+    <parent link="robot_base"/>
+    <child link="${prefix}base_link"/>
     <origin xyz="0 0 0" rpy="0 0 0"/>
   </joint>
-  <!-- پایه موقت ربات -->
-  <link name="base_link">
-    <visual>
-      <geometry>
-        <box size="0.3 0.3 0.2"/>
-      </geometry>
-    </visual>
-    <collision>
-      <geometry>
-        <box size="0.3 0.3 0.2"/>
-      </geometry>
-    </collision>
-    <inertial>
-      <mass value="10.0"/>
-      <origin xyz="0 0 0"/>
-      <inertia
-        ixx="0.1"
-        ixy="0.0"
-        ixz="0.0"
-        iyy="0.1"
-        iyz="0.0"
-        izz="0.1"/>
-    </inertial>
-  </link>
-  <joint name="robot_base_to_base_link" type="fixed">
-    <parent link="robot_base"/>
-    <child link="base_link"/>
-    <origin xyz="0 0 0.1" rpy="0 0 0"/>
+  <!-- The TCP is configurable because it belongs to the future end effector. -->
+  <link name="gripper_tcp"/>
+  <joint name="tool0_to_gripper_tcp" type="fixed">
+    <parent link="${prefix}tool0"/>
+    <child link="gripper_tcp"/>
+    <origin xyz="$(arg tcp_xyz)" rpy="$(arg tcp_rpy)"/>
   </joint>
-  <!-- محل ابزار ربات -->
-  <link name="tool0"/>
-  <joint name="base_to_tool" type="fixed">
-    <parent link="base_link"/>
-    <child link="tool0"/>
-    <origin xyz="0 0 0.5" rpy="0 0 0"/>
-  </joint>
-  <!-- محل TCP گریپر -->
-  <link name="gripper_tcp"/>
-  <joint name="tool_to_gripper_tcp" type="fixed">
-    <parent link="tool0"/>
-    <child link="gripper_tcp"/>
-    <origin xyz="0 0 0.1" rpy="0 0 0"/>
-  </joint>
-  <!-- محل نصب دوربین -->
   <link name="front_camera_link"/>
   <joint name="cell_to_front_camera" type="fixed">
@@ -69,12 +48,10 @@
     <origin xyz="1.0 0 1.8" rpy="0 0 0"/>
   </joint>
-  <!-- Optical frame دوربین -->
   <link name="front_camera_optical_frame"/>
   <joint name="camera_to_optical" type="fixed">
     <parent link="front_camera_link"/>
     <child link="front_camera_optical_frame"/>
-    <origin xyz="0 0 0" rpy="-1.5708 0 -1.5708"/>
+    <origin xyz="0 0 0" rpy="-1.57079632679 0 -1.57079632679"/>
   </joint>
-  <!-- فریم محل جعبه یا Bin -->
   <link name="bin_frame"/>
   <joint name="cell_to_bin" type="fixed">

Commit message: Add RViz robot and target visualization

File: src/foundation/pickcell_description/urdf/pickcell.urdf.xacro (robot description, xacro)
@@ -54,9 +54,3 @@
     <origin xyz="0 0 0" rpy="-1.57079632679 0 -1.57079632679"/>
   </joint>
-  <link name="bin_frame"/>
-  <joint name="cell_to_bin" type="fixed">
-    <parent link="cell"/>
-    <child link="bin_frame"/>
-    <origin xyz="0.8 0 0" rpy="0 0 0"/>
-  </joint>
 </robot>

Commit message: Configure KR 180 cell with loaded box

File: src/foundation/pickcell_description/urdf/pickcell.urdf.xacro (robot description, xacro)
@@ -2,9 +2,10 @@
 <robot xmlns:xacro="http://www.ros.org/wiki/xacro" name="pickcell">
   <!--
-    Cell description using the maintained ROS 2 model of the KUKA
-    KR 16 R2010-2. Robot dimensions, joint axes, joint limits and meshes live
-    in kuka_cybertech_support; they are intentionally not duplicated here.
+    Cell description configured for a KUKA KR 180 R2900-2. The maintained
+    KR 240 R2900-2 ROS model is used as a temporary same-family, same-reach
+    geometry proxy until an exact KR 180 mesh package is available.
   -->
-  <xacro:include filename="$(find kuka_cybertech_support)/urdf/kr16_r2010_2_macro.xacro"/>
+  <xacro:include filename="$(find kuka_quantec_support)/urdf/kr240_r2900_2_macro.xacro"/>
+  <xacro:include filename="$(find pickcell_description)/urdf/chemical_bag.xacro"/>
   <xacro:arg name="robot_prefix" default=""/>
   <xacro:arg name="robot_mount_xyz" default="0 0 0"/>
@@ -13,4 +14,22 @@
   <xacro:arg name="tcp_rpy" default="0 0 0"/>
   <xacro:property name="prefix" value="$(arg robot_prefix)"/>
+  <material name="wood_brown">
+    <color rgba="0.55 0.30 0.12 1.0"/>
+  </material>
+  <xacro:macro name="wooden_box_panel" params="xyz size">
+    <visual>
+      <origin xyz="${xyz}" rpy="0 0 0"/>
+      <geometry>
+        <box size="${size}"/>
+      </geometry>
+      <material name="wood_brown"/>
+    </visual>
+    <collision>
+      <origin xyz="${xyz}" rpy="0 0 0"/>
+      <geometry>
+        <box size="${size}"/>
+      </geometry>
+    </collision>
+  </xacro:macro>
   <link name="world"/>
   <link name="cell"/>
@@ -27,7 +46,55 @@
     <origin xyz="$(arg robot_mount_xyz)" rpy="$(arg robot_mount_rpy)"/>
   </joint>
-  <xacro:kuka_kr16_r2010_2_robot
+  <!-- Open wooden box: 0.8 m deep, 1.2 m wide, 0.8 m high, with 30 mm
+       bottom/walls and no top panel. Its nearest outer face is 1.0 m in front
+       of the robot base. -->
+  <link name="wooden_box">
+    <!-- Bottom: top surface is 30 mm above the floor. -->
+    <xacro:wooden_box_panel xyz="0 0 -0.385" size="0.8 1.2 0.03"/>
+    <!-- Front and rear walls. -->
+    <xacro:wooden_box_panel xyz="-0.385 0 0" size="0.03 1.2 0.8"/>
+    <xacro:wooden_box_panel xyz="0.385 0 0" size="0.03 1.2 0.8"/>
+    <!-- Side walls fit between the front and rear walls. -->
+    <xacro:wooden_box_panel xyz="0 -0.585 0" size="0.74 0.03 0.8"/>
+    <xacro:wooden_box_panel xyz="0 0.585 0" size="0.74 0.03 0.8"/>
+  </link>
+  <joint name="cell_to_wooden_box" type="fixed">
+    <parent link="cell"/>
+    <child link="wooden_box"/>
+    <origin xyz="1.4 0 0.4" rpy="0 0 0"/>
+  </joint>
+  <!-- Repeatable randomized stack of filled chemical bags. Coordinates are
+       relative to the box centre; small gaps avoid initial self-collisions. -->
+  <xacro:chemical_bag parent="wooden_box" name="chemical_bag_01"
+    xyz="-0.025 -0.245 -0.285" rpy="0 0 0.035"
+    mass="22.4" scale_x="0.97" scale_y="1.02" scale_z="1.00"/>
+  <xacro:chemical_bag parent="wooden_box" name="chemical_bag_02"
+    xyz="0.030 0.250 -0.285" rpy="0 0 -0.045"
+    mass="23.1" scale_x="1.01" scale_y="0.96" scale_z="0.98"/>
+  <xacro:chemical_bag parent="wooden_box" name="chemical_bag_03"
+    xyz="0.018 -0.238 -0.120" rpy="0 0 -0.055"
+    mass="21.8" scale_x="0.98" scale_y="1.01" scale_z="1.00"/>
+  <xacro:chemical_bag parent="wooden_box" name="chemical_bag_04"
+    xyz="-0.032 0.242 -0.120" rpy="0 0 0.050"
+    mass="23.6" scale_x="1.00" scale_y="0.97" scale_z="0.99"/>
+  <xacro:chemical_bag parent="wooden_box" name="chemical_bag_05"
+    xyz="-0.035 -0.250 0.045" rpy="0 0 0.060"
+    mass="22.7" scale_x="0.96" scale_y="1.03" scale_z="1.00"/>
+  <xacro:chemical_bag parent="wooden_box" name="chemical_bag_06"
+    xyz="0.025 0.235 0.045" rpy="0 0 -0.030"
+    mass="21.5" scale_x="1.02" scale_y="0.95" scale_z="0.97"/>
+  <xacro:chemical_bag parent="wooden_box" name="chemical_bag_07"
+    xyz="0.032 -0.240 0.210" rpy="0 0 -0.040"
+    mass="23.3" scale_x="0.99" scale_y="1.00" scale_z="0.98"/>
+  <xacro:chemical_bag parent="wooden_box" name="chemical_bag_08"
+    xyz="-0.020 0.248 0.210" rpy="0 0 0.055"
+    mass="22.0" scale_x="0.97" scale_y="1.02" scale_z="1.00"/>
+  <!-- The final bag rises about 5 cm above the 0.8 m rim. -->
+  <xacro:chemical_bag parent="wooden_box" name="chemical_bag_09"
+    xyz="0.015 0.005 0.375" rpy="0 0 -0.025"
+    mass="22.9" scale_x="1.00" scale_y="0.98" scale_z="1.00"/>
+  <xacro:kuka_kr240_r2900_2_robot
     prefix="${prefix}"
-    package_name="kuka_cybertech_support"/>
+    package_name="kuka_quantec_support"/>
   <joint name="robot_base_to_kuka_base_link" type="fixed">
     <parent link="robot_base"/>

Commit message: Separate pallet scene from robot visualization
Replace the loaded box with a reusable wall-free pallet model and keep it in the complete URDF for collision checking. Add a pallet-only description, an overhead depth-camera frame, and independent RViz displays for the robot, pallet load, and simulated point cloud.

File: src/foundation/pickcell_description/urdf/pickcell.urdf.xacro (robot description, xacro)
@@ -7,5 +7,5 @@
   -->
   <xacro:include filename="$(find kuka_quantec_support)/urdf/kr240_r2900_2_macro.xacro"/>
-  <xacro:include filename="$(find pickcell_description)/urdf/chemical_bag.xacro"/>
+  <xacro:include filename="$(find pickcell_description)/urdf/bag_pallet.xacro"/>
   <xacro:arg name="robot_prefix" default=""/>
   <xacro:arg name="robot_mount_xyz" default="0 0 0"/>
@@ -13,23 +13,6 @@
   <xacro:arg name="tcp_xyz" default="0 0 0"/>
   <xacro:arg name="tcp_rpy" default="0 0 0"/>
+  <xacro:arg name="include_pallet" default="true"/>
   <xacro:property name="prefix" value="$(arg robot_prefix)"/>
-  <material name="wood_brown">
-    <color rgba="0.55 0.30 0.12 1.0"/>
-  </material>
-  <xacro:macro name="wooden_box_panel" params="xyz size">
-    <visual>
-      <origin xyz="${xyz}" rpy="0 0 0"/>
-      <geometry>
-        <box size="${size}"/>
-      </geometry>
-      <material name="wood_brown"/>
-    </visual>
-    <collision>
-      <origin xyz="${xyz}" rpy="0 0 0"/>
-      <geometry>
-        <box size="${size}"/>
-      </geometry>
-    </collision>
-  </xacro:macro>
   <link name="world"/>
   <link name="cell"/>
@@ -46,52 +29,9 @@
     <origin xyz="$(arg robot_mount_xyz)" rpy="$(arg robot_mount_rpy)"/>
   </joint>
-  <!-- Open wooden box: 0.8 m deep, 1.2 m wide, 0.8 m high, with 30 mm
-       bottom/walls and no top panel. Its nearest outer face is 1.0 m in front
-       of the robot base. -->
-  <link name="wooden_box">
-    <!-- Bottom: top surface is 30 mm above the floor. -->
-    <xacro:wooden_box_panel xyz="0 0 -0.385" size="0.8 1.2 0.03"/>
-    <!-- Front and rear walls. -->
-    <xacro:wooden_box_panel xyz="-0.385 0 0" size="0.03 1.2 0.8"/>
-    <xacro:wooden_box_panel xyz="0.385 0 0" size="0.03 1.2 0.8"/>
-    <!-- Side walls fit between the front and rear walls. -->
-    <xacro:wooden_box_panel xyz="0 -0.585 0" size="0.74 0.03 0.8"/>
-    <xacro:wooden_box_panel xyz="0 0.585 0" size="0.74 0.03 0.8"/>
-  </link>
-  <joint name="cell_to_wooden_box" type="fixed">
-    <parent link="cell"/>
-    <child link="wooden_box"/>
-    <origin xyz="1.4 0 0.4" rpy="0 0 0"/>
-  </joint>
-  <!-- Repeatable randomized stack of filled chemical bags. Coordinates are
-       relative to the box centre; small gaps avoid initial self-collisions. -->
-  <xacro:chemical_bag parent="wooden_box" name="chemical_bag_01"
-    xyz="-0.025 -0.245 -0.285" rpy="0 0 0.035"
-    mass="22.4" scale_x="0.97" scale_y="1.02" scale_z="1.00"/>
-  <xacro:chemical_bag parent="wooden_box" name="chemical_bag_02"
-    xyz="0.030 0.250 -0.285" rpy="0 0 -0.045"
-    mass="23.1" scale_x="1.01" scale_y="0.96" scale_z="0.98"/>
-  <xacro:chemical_bag parent="wooden_box" name="chemical_bag_03"
-    xyz="0.018 -0.238 -0.120" rpy="0 0 -0.055"
-    mass="21.8" scale_x="0.98" scale_y="1.01" scale_z="1.00"/>
-  <xacro:chemical_bag parent="wooden_box" name="chemical_bag_04"
-    xyz="-0.032 0.242 -0.120" rpy="0 0 0.050"
-    mass="23.6" scale_x="1.00" scale_y="0.97" scale_z="0.99"/>
-  <xacro:chemical_bag parent="wooden_box" name="chemical_bag_05"
-    xyz="-0.035 -0.250 0.045" rpy="0 0 0.060"
-    mass="22.7" scale_x="0.96" scale_y="1.03" scale_z="1.00"/>
-  <xacro:chemical_bag parent="wooden_box" name="chemical_bag_06"
-    xyz="0.025 0.235 0.045" rpy="0 0 -0.030"
-    mass="21.5" scale_x="1.02" scale_y="0.95" scale_z="0.97"/>
-  <xacro:chemical_bag parent="wooden_box" name="chemical_bag_07"
-    xyz="0.032 -0.240 0.210" rpy="0 0 -0.040"
-    mass="23.3" scale_x="0.99" scale_y="1.00" scale_z="0.98"/>
-  <xacro:chemical_bag parent="wooden_box" name="chemical_bag_08"
-    xyz="-0.020 0.248 0.210" rpy="0 0 0.055"
-    mass="22.0" scale_x="0.97" scale_y="1.02" scale_z="1.00"/>
-  <!-- The final bag rises about 5 cm above the 0.8 m rim. -->
-  <xacro:chemical_bag parent="wooden_box" name="chemical_bag_09"
-    xyz="0.015 0.005 0.375" rpy="0 0 -0.025"
-    mass="22.9" scale_x="1.00" scale_y="0.98" scale_z="1.00"/>
+  <!-- Kept in the complete model for MoveIt collision checking, but omitted
+       from the robot-only description consumed by RViz. -->
+  <xacro:if value="$(arg include_pallet)">
+    <xacro:bag_pallet parent="cell"/>
+  </xacro:if>
   <xacro:kuka_kr240_r2900_2_robot
     prefix="${prefix}"
@@ -109,14 +49,16 @@
     <origin xyz="$(arg tcp_xyz)" rpy="$(arg tcp_rpy)"/>
   </joint>
-  <link name="front_camera_link"/>
-  <joint name="cell_to_front_camera" type="fixed">
+  <!-- Fixed overhead depth camera. Its optical +Z axis points straight down
+       at the pallet centre, matching the ROS optical-frame convention. -->
+  <link name="overhead_depth_camera_link"/>
+  <joint name="cell_to_overhead_depth_camera" type="fixed">
     <parent link="cell"/>
-    <child link="front_camera_link"/>
-    <origin xyz="1.0 0 1.8" rpy="0 0 0"/>
+    <child link="overhead_depth_camera_link"/>
+    <origin xyz="1.4 0 2.0" rpy="0 1.57079632679 0"/>
   </joint>
-  <link name="front_camera_optical_frame"/>
-  <joint name="camera_to_optical" type="fixed">
-    <parent link="front_camera_link"/>
-    <child link="front_camera_optical_frame"/>
+  <link name="overhead_depth_camera_optical_frame"/>
+  <joint name="overhead_depth_camera_to_optical" type="fixed">
+    <parent link="overhead_depth_camera_link"/>
+    <child link="overhead_depth_camera_optical_frame"/>
     <origin xyz="0 0 0" rpy="-1.57079632679 0 -1.57079632679"/>
   </joint>

Commit message: Add planned repeating pick-place motion demo

File: src/foundation/pickcell_description/urdf/pickcell.urdf.xacro (robot description, xacro)
@@ -9,4 +9,5 @@
   <xacro:include filename="$(find pickcell_description)/urdf/bag_pallet.xacro"/>
   <xacro:include filename="$(find pickcell_description)/urdf/drop_box.xacro"/>
+  <xacro:include filename="$(find pickcell_description)/urdf/simple_gripper.xacro"/>
   <xacro:arg name="robot_prefix" default=""/>
   <xacro:arg name="robot_mount_xyz" default="0 0 0"/>
@@ -47,11 +48,6 @@
     <origin xyz="0 0 0" rpy="0 0 0"/>
   </joint>
-  <!-- The TCP is configurable because it belongs to the future end effector. -->
-  <link name="gripper_tcp"/>
-  <joint name="tool0_to_gripper_tcp" type="fixed">
-    <parent link="${prefix}tool0"/>
-    <child link="gripper_tcp"/>
-    <origin xyz="$(arg tcp_xyz)" rpy="$(arg tcp_rpy)"/>
-  </joint>
+  <xacro:simple_gripper parent="${prefix}tool0"
+    tcp_xyz="$(arg tcp_xyz)" tcp_rpy="$(arg tcp_rpy)"/>
   <!-- Fixed overhead depth camera. Its optical +Z axis points straight down
        at the pallet centre, matching the ROS optical-frame convention. -->
