Commit message: Configure two-anchor simulation and display

File: src/foundation/pickcell_description/urdf/bag_pallet.xacro (robot description, xacro)
@@ -2,5 +2,5 @@
 <robot xmlns:xacro="http://www.ros.org/wiki/xacro">
   <xacro:include filename="$(find pickcell_description)/urdf/chemical_bag.xacro"/>
-  <xacro:macro name="bag_pallet" params="parent">
+  <xacro:macro name="bag_pallet" params="parent include_bags:=true">
     <!-- Wall-free wooden pallet: 0.8 m deep, 1.2 m wide and 0.15 m high. -->
     <link name="bag_pallet">
@@ -24,5 +24,7 @@
       <origin xyz="1.4 0 0.075" rpy="0 0 0"/>
     </joint>
-    <!-- Repeatable randomized five-layer stack. -->
+    <!-- Repeatable randomized five-layer stack. Stateful runtime bags are
+         excluded from MoveIt, where fixed links would become stale. -->
+    <xacro:if value="${include_bags}">
     <xacro:chemical_bag parent="bag_pallet" name="chemical_bag_01"
       xyz="-0.025 -0.245 0.155" rpy="0 0 0.035"
@@ -52,4 +54,5 @@
       xyz="0.015 0.005 0.815" rpy="0 0 -0.025"
       mass="22.9" scale_x="1.00" scale_y="0.98" scale_z="1.00"/>
+    </xacro:if>
   </xacro:macro>
 </robot>

File: src/foundation/pickcell_description/urdf/pickcell.urdf.xacro (robot description, xacro)
@@ -16,4 +16,5 @@
   <xacro:arg name="tcp_rpy" default="0 0 0"/>
   <xacro:arg name="include_pallet" default="true"/>
+  <xacro:arg name="include_bags" default="true"/>
   <xacro:arg name="include_drop_box" default="true"/>
   <xacro:property name="prefix" value="$(arg robot_prefix)"/>
@@ -35,5 +36,5 @@
        from the robot-only description consumed by RViz. -->
   <xacro:if value="$(arg include_pallet)">
-    <xacro:bag_pallet parent="cell"/>
+    <xacro:bag_pallet parent="cell" include_bags="$(arg include_bags)"/>
   </xacro:if>
   <xacro:if value="$(arg include_drop_box)">
